File: catt_jtag.kicad_pcb (KiCad board)
At the start: 2 copper layers, 16 x 20 mm, 7 parts, among them J1 CATT, J2 JTAG, J3 I2C

Commit message: Choose new components
Other:
- board text added: "This side should face the back of the device"
- board text removed: "This side should face to the back of the device"
Changed lines of the file:
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@@
 			)
 		)
-		(property "Datasheet" "https://www.lcsc.com/product-detail/Chip-Resistor-Surface-Mount_UNI-ROYAL-Uniroyal-Elec-0402WGF2201TCE_C25879.html"
+		(property "Datasheet" "https://jlcpcb.com/partdetail/12256-0402WGF1001TCE/C11702"
 			(at 0 0 90)
 			(unlocked yes)
@@
 		)
 		(property ki_fp_filters "R_*")
-		(sheetname "Root")
+		(sheetname "/")
 		(sheetfile "catt_jtag.kicad_sch")
 		(attr smd)
@@
 			)
 		)
-		(property "Datasheet" "https://www.lcsc.com/product-detail/Chip-Resistor-Surface-Mount_UNI-ROYAL-Uniroyal-Elec-0402WGF2201TCE_C25879.html"
+		(property "Datasheet" "https://jlcpcb.com/partdetail/12256-0402WGF1001TCE/C11702"
 			(at 0 0 90)
 			(unlocked yes)
@@
 		)
 		(property ki_fp_filters "R_*")
-		(sheetname "Root")
+		(sheetname "/")
 		(sheetfile "catt_jtag.kicad_sch")
 		(attr smd)
@@
 			)
 		)
-		(property "Datasheet" "https://datasheet.lcsc.com/lcsc/2402181501_XINGLIGHT-XL-1608UVC-04_C7371898.pdf"
+		(property "Datasheet" "https://jlcpcb.com/partdetail/C7496820"
 			(at 0 0 90)
 			(unlocked yes)
@@
 			)
 		)
-		(property "LCSC" "C7371898"
+		(property "LCSC" "C7496820"
 			(at 0 0 90)
 			(unlocked yes)
@@
 		)
 		(property ki_fp_filters "LED* LED_SMD:* LED_THT:*")
-		(sheetname "Root")
+		(sheetname "/")
 		(sheetfile "catt_jtag.kicad_sch")
 		(attr smd)
@@
 			)
 		)
-		(property "Datasheet" "https://datasheet.lcsc.com/lcsc/1811151533_JST-Sales-America-SM04B-SRSS-TB-LF-SN_C160404.pdf"
+		(property "Datasheet" "https://jlcpcb.com/partdetail/HongCheng-HCZZ00324/C7433425"
 			(at 0 0 90)
 			(layer "F.Fab")
@@
 			)
 		)
-		(property "LCSC" "C160404"
+		(property "LCSC" "C7433425"
 			(at 0 0 270)
 			(unlocked yes)
@@
 		)
 		(property ki_fp_filters "*1X04_1MM_RA* *1X04_1MM_RA_STRESSRELIEF*")
-		(sheetname "Root")
+		(sheetname "/")
 		(sheetfile "catt_jtag.kicad_sch")
 		(attr smd)
@@
 			)
 		)
-		(property "Datasheet" "https://www.lcsc.com/product-detail/Pin-Headers_Yxcon-P125-1207A0BR138A1_C19190502.html"
+		(property "Datasheet" "https://jlcpcb.com/partdetail/Xfcn-PZ254R_1214P/C492435"
 			(at 0 0 0)
 			(unlocked yes)
@@
 			)
 		)
-		(property "LCSC" "C19190502"
+		(property "LCSC" "C492435"
 			(at 0 0 0)
 			(unlocked yes)
@@
 		)
 		(property ki_fp_filters "Connector*:*_2x??_*")
-		(sheetname "Root")
+		(sheetname "/")
 		(sheetfile "catt_jtag.kicad_sch")
 		(attr through_hole)
@@
 			)
 		)
-		(property "Datasheet" "https://jlcpcb.com/partdetail/Wcon-313010SG0BK00T1/C783829"
+		(property "Datasheet" "https://jlcpcb.com/partdetail/Hanxia-HX_JN1_27_2x5P_ZZ_H49/C42372547"
 			(at 0 0 90)
 			(layer "F.Fab")
@@
 			)
 		)
-		(property "LCSC" "C783829"
+		(property "LCSC" "C42372547"
 			(at 0 0 270)
 			(unlocked yes)
@@
 		)
 		(property ki_fp_filters "PinHeader?2x05?P1.27mm*")
-		(sheetname "Root")
+		(sheetname "/")
 		(sheetfile "catt_jtag.kicad_sch")
 		(attr through_hole)
@@
 			)
 		)
-		(property "Datasheet" "https://www.lcsc.com/product-detail/Chip-Resistor-Surface-Mount_UNI-ROYAL-Uniroyal-Elec-0402WGF2201TCE_C25879.html"
+		(property "Datasheet" "https://jlcpcb.com/partdetail/12256-0402WGF1001TCE/C11702"
 			(at 0 0 270)
 			(unlocked yes)
@@
 		)
 		(property ki_fp_filters "R_*")
-		(sheetname "Root")
+		(sheetname "/")
 		(sheetfile "catt_jtag.kicad_sch")
 		(attr smd)
@@
 		(layer "Edge.Cuts")
 	)
-	(gr_text "This side should face to\nthe back of the device"
+	(gr_text "This side should face\nthe back of the device"
 		(at 6.5 0 90)
 		(layer "B.SilkS")
